File: uino-1284p.brd (EAGLE design)
At the start: 68.6 x 53.3 mm, 59 parts, among them J1 POWER, J2 POWER_JACKPTH, J4 POWER_SELECT, J6 IO, J7 ANALOG, J8 IOL, J9 IOH, U1 LD117AS50TR, U2 ATMEGA1284AU, U3 ATMEGA8U2AU, X1 16MHz, X2 16MHz

Commit message: Unified device name text on board. Arranged name labels.
Parts:
- renumbered LED1 to E1, LED2 to E2, LED3 to E3, LED4 to E4, LED5 to E5
Other:
- board text added: "v0.4 2016/11/03"
- board text removed: "v0.3 2011/12/31"

Commit message: Changed to micro USB. Moved USB ICSP header.
Parts:
- removed J6: IO, adilinden:2X05
- removed U3: ATMEGA8U2AU, SparkFun:TQFP32-08
- removed USB: MINI-USB-SHIELD-UX60-MB-5ST, adafruit:USB-MINIB
- added IC1: LD117AS50TR, adilinden:SOT223
- added JP1: POWER, SparkFun:1X06
- added JP5: POWER_SELECT, SparkFun:1X03
- C1: value 0.01u -> 0.1u
- C11, C12, C2, C3: value 0.1u -> 22p
- C14, C17: value 22p -> 0.1u
- C15, C16: value 22p -> 10u; device rcl:C0805 -> rcl:CT3216
- C20: value 1u -> 0.1u
- C4: value 0.1u -> 1u
- C5: value 10u -> 0.01u; device rcl:CT3216 -> rcl:C0805
- C6: value 10u -> 0.1u; device rcl:CT3216 -> rcl:C0805
- J1: value POWER -> Micro USB; device SparkFun:1X06 -> adi-misc:ZX62D-AB-5P8
- J2: value POWER_JACKPTH -> M03X2; device SparkFun:POWER_JACK_PTH -> adi-misc:2X03
- J3: device adilinden:2X03 -> SparkFun:POWER_JACK_PTH
- J4: value POWER_SELECT -> M03X2; device SparkFun:1X03 -> adi-misc:2X03
- J5: value (none) -> IO; device adilinden:2X03 -> adilinden:2X05
- R1: value 22 -> 1k
- R2: value 22 -> 10k
- R3, R4: value 1k -> 22
- R5: value 1k -> 10k
- R6, R7: value 10k -> 1k
- U1: value LD117AS50TR -> ATMEGA8U2AU; device adilinden:SOT223 -> SparkFun:TQFP32-08
- moved J3 71.0 mm to (-3.17, 7.62)
- moved C11 51.5 mm to (59.8, 25.8), turned to 90 degrees
- moved J4 51.2 mm to (64.9, 27.9), turned to 270 degrees
- moved R7 51.0 mm to (9.53, 21.0), turned to 0 degrees
- moved J1 47.3 mm to (1.78, 38.1), turned to 270 degrees
- moved J2 40.2 mm to (19.7, 40.6), turned to 0 degrees
- moved C8 38.4 mm to (9.53, 14.6), turned to 180 degrees
- moved J5 38.4 mm to (22.9, 3.81)
- moved C15 37.0 mm to (22.9, 22.2), turned to 90 degrees
- moved C20 36.6 mm to (55.9, 16.9)
- moved C14 34.0 mm to (26.0, 22.2)
- moved R5 31.4 mm to (31.8, 39.4), turned to 270 degrees
- moved C9 29.1 mm to (26.7, 8.26), turned to 0 degrees
- moved R10 28.6 mm to (57.8, 37.5)
- moved X1 25.6 mm to (31.8, 29.6), turned to 90 degrees
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- renumbered E1 to LED2, E2 to LED4, E3 to LED1, E4 to LED3, E5 to LED5, J7 to JP2, J8 to JP3, J9 to JP4, PAD1 to SJ1, U2 to IC2
Connections:
- net 3V3: now also JP1.2; no longer J1.2
- net A6: now also J5.9; no longer J6.9
- net A7: now also J5.10; no longer J6.10
- net AREF: now also C13.1; no longer C18.1
- net D+: now also R4.2, U1.29; no longer R1.2, U3.29
- net D-: now also R3.2, U1.30; no longer R2.2, U3.30
- net D0: now also R11.1; no longer R12.1
- net D1: now also R12.1; no longer R11.1
- net D18: now also J5.3; no longer J6.3
- net D19: now also J5.4; no longer J6.4
- net D20: now also J5.5; no longer J6.5
- net D21: now also J5.6; no longer J6.6
- net D22: now also J5.7; no longer J6.7
- net D23: now also J5.8; no longer J6.8
- net EVCC: now also C14.1, C15.+, IC1.2, IC1.4, JP5.1; no longer C4.1, C5.+, J4.1, U1.2, U1.4
- net GND: now also C15.-, C16.-, C19.2, C5.2, C6.2, IC1.1, J1.S1, J1.S2, J2.6, J3.GND, J3.GNDBREAK, J4.6, JP1.4, JP1.5, R5.1, U1.28, U1.3; no longer C15.2, C16.2, C5.-, C6.-, C7.2, J1.4, J2.GND, J2.GNDBREAK, J3.6, J5.6, R10.1, U1.1, U3.28, U3.3, USB.GND
- net L1: now also J5.1, R6.2; no longer J6.1, R3.2
- net L2: now also J5.2, R8.2; no longer J6.2, R4.2
- net MISO: now also J4.1; no longer J3.1
- net MOSI: now also J4.4; no longer J3.4
- net N$10: now also C4.1, U1.27; no longer C20.1, U3.27
- net N$11: now also R6.1; no longer R3.1
- net N$12: now also R8.1; no longer R4.1
- net N$13: now also J2.1, U1.17; no longer J5.1, U3.17
- net N$14: now also J2.3, U1.15; no longer J5.3, U3.15
- net N$15: now also J2.5, R2.1, U1.24; no longer J5.5, R6.1, U3.24
- net N$16: now also J2.4, U1.16; no longer J5.4, U3.16
- net N$2: now also C5.1; no longer C1.1
- net N$23: now also C11.1, X2.P$2; no longer C14.1, X1.P$2
- net N$24: now also C12.1, X2.P$1; no longer C15.1, X1.P$1
- net N$25: now also J3.PWR; no longer J2.PWR
- net N$26: now also R7.1; no longer R8.1
- net N$29: now also U1.10; no longer U3.10
- net N$3: now also C7.1; no longer C19.1
- net N$30: now also U1.11; no longer U3.11
- net N$31: now also C7.2, R5.2, U1.13; no longer C19.2, R10.2, U3.13
- net N$34: now also R1.1; no longer R5.1
- net N$4: now also J1.2, R3.1; no longer R2.1, USB.D-
- net N$5: now also J1.3, R4.1; no longer R1.1, USB.D+
- net N$6: now also R11.2, U1.9; no longer R12.2, U3.9
- net N$7: now also R12.2, U1.8; no longer R11.2, U3.8
- net N$8: now also C2.1, U1.1, X1.P$2; no longer C16.1, U3.1, X2.P$2
- net N$9: now also C3.1, U1.2, X1.P$1; no longer C17.1, U3.2, X2.P$1
- net RESET: now also J4.5, JP1.1, R10.1; no longer J1.1, J3.5, R7.1
- net SCK: now also J4.3; no longer J3.3
- net UVCC: now also C6.1, JP5.3, U1.31; no longer C2.1, J4.3, U3.31
- net VBUS: now also J1.1; no longer USB.VBUS
- net VCC: now also C1.1, C16.+, C17.1, C18.1, C19.1, C20.1, J2.2, JP1.3, JP5.2, R1.2, R10.2, R2.2, U1.32, U1.4; no longer C11.1, C12.1, C13.1, C6.+, C7.1, C9.1, J1.3, J3.2, J5.2, R5.2, R6.2, R8.2, U3.32, U3.4
- net VIN: now also C9.1, IC1.3, JP1.6; no longer C3.1, J1.6, U1.3
Routing:
- net GND: track 4.01 -> 7.43 mm, vias 47 -> 50
- net D+: track 15.1 -> 18.4 mm
- net D-: track 17.3 -> 20.6 mm
- net N$2: track 15.7 -> 19.0 mm
- net N$31: track 8.37 -> 11.0 mm
- net N$3: track 17.2 -> 19.8 mm
- net N$14: track 7.10 -> 4.71 mm
- net N$16: track 10.0 -> 8.01 mm
- net VCC: track 191.5 -> 190.0 mm
- net N$13: track 8.10 -> 6.71 mm
- net N$5: track 9.07 -> 7.91 mm
- net N$15: track 18.2 -> 19.2 mm
- net N$4: track 6.86 -> 6.16 mm
Other:
- board text added: "v1.0 2016/11/03"
- board text removed: "v0.4 2016/11/03"
